File: hardware/nfc.kicad_pcb (KiCad board)
At the start: 2 copper layers, 80 x 50 mm, 63 parts, among them J1 CONN_01X03, P1 CON-SENSOR2, P2 BOOT, P3 DEBUG, U1 XMC130024, U2 PN7150, U3 DRILL, U4 DRILL, U5 DRILL, U6 DRILL, U7 DRILL, U8 DRILL, X1 27.12MHZ

Commit message: add datamatrix position
Parts:
- added REF**: 5x5 Datamatrix, kicad-libraries:5x5 Datamatrix, B.Cu at (181.3, 93.0)
Other:
- net class Default removed
